File: PCB/KiCad/Keypad.sch (KiCad schematic (older format))
At the start: 17 parts, among them SW1 SW_SPDT, U1 TP4056, U2 MT3608, U3 WeMos_D1_mini

Commit message: kicad files updated.
Parts:
- removed Keypad1: Conn_01x09, Connector_PinHeader_2.54mm:PinHeader_1x09_P2.54mm_Vertical, symbol Connector_Generic:Conn_01x09
- removed SW1: SW_SPDT, Button_Switch_THT:SW_Slide_1P2T_CK_OS102011MS2Q, symbol Switch:SW_SPDT
- added Keypad1: Conn_01x03, Connector_PinHeader_2.54mm:PinHeader_1x03_P2.54mm_Vertical, symbol Connector_Generic:Conn_01x03
- added R6: 500K, Resistor_THT:R_Axial_DIN0207_L6.3mm_D2.5mm_P10.16mm_Horizontal, symbol Device:R
- added SW1: SW_DIP_x01, Keypad:Mini_Latching_Torch_Switch, symbol Switch:SW_DIP_x01
- added U4: MCP3421A0T-ECH, Package_TO_SOT_SMD:SOT-23-6_Handsoldering, symbol Analog_ADC:MCP3421A0T-ECH
- R5: value 100k -> 560k
Connections:
- net +3V3: now also Keypad1.3 (Pin_3), U4.5 (Vdd); no longer R1.1
- net GND: now also D1.1 (K), D2.1 (K), Keypad1.2 (Pin_2), R6.2, U4.2 (Vss), U4.6 (Vin-)
- net SCL: now also U4.3 (SCL)
- net SDA: now also U4.4 (SDA)
- net V+1: now also SW1.1
- net V+2: no longer U2.1 (V_IN+)
- net at R5.2: now also R6.1, U4.1 (Vin+); no longer U3.2 (A0)
- net KP1: no longer names the net of U3.11 (D4)
- net KP2: no longer names the net of U3.12 (D3)
- net KP3 renamed green
- net green: now also R3.1
- net KP4 renamed yellow
- net yellow: now also R2.1
- net KP5 renamed red
- net red: now also R1.1
- net KP6: no longer names the net of U3.4 (SCK/D5)
- net KP7: no longer names the net of U3.3 (D0)
- removed net LED_Control1: D1.1 (K), R2.1, U3.16 (TX)
- removed net LED_Control2: D2.1 (K), R3.1, U3.15 (RX)
- new net: SW1.2, U2.1 (V_IN+)
- new net keypad: Keypad1.1 (Pin_1), U3.2 (A0)
- no-connect marks 6 -> 9
Other:
- note added: "Analog -> Digital I2C Converter"
- note added: "LED Icons (Optional)"
- note added: "Power Conversion / Battery Management"
- moved on the sheet: D1, D2, D3, R1, R2, R3, R5, U2
